File: pan-ard-inf/kicad/pan-ard-inf.kicad_pcb (KiCad board)
At the start: 2 copper layers, 101.6 x 53.3 mm, 49 parts, among them J1 Power, J10 PJ-037B, J2 Analog, J3 Analog, J4 Digital, J5 PWM, J6 PWM, J7 Communication, J8 SJ1-3534N, J9 SJ1-3534N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

Commit message: updated kicad files
Parts:
- J3: value Analog -> type="I" model="Analog" lib=""
