File: pan-ard-inf/kicad/pan-ard-inf.kicad_sch (KiCad schematic)
At the start: 52 parts, among them J1 Power, J10 PJ-037B, J2 Analog, J3 Analog, J4 Digital, J5 PWM, J6 PWM, J7 Communication, J8 SJ1-3534N, J9 SJ1-3534N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

Commit message: updated kicad files
Parts:
- I1, I2: Spice_Model dc 0 ac 1.27m sin(0 1.27m 60) -> (none); Spice_Netlist_Enabled Y -> (none); Spice_Primitive I -> (none)
- J1: Spice_Model Power -> (none); Spice_Netlist_Enabled N -> (none); Spice_Primitive J -> (none)
- J10: Spice_Model Barrel_Jack -> (none); Spice_Netlist_Enabled N -> (none); Spice_Primitive J -> (none)
- J2: Spice_Model Analog -> (none); Spice_Netlist_Enabled N -> (none); Spice_Primitive J -> (none)
- J3: value Analog -> ${SIM.PARAMS}; Spice_Netlist_Enabled N -> (none); Spice_Primitive I -> (none)
- J4: Spice_Model Digital -> (none); Spice_Netlist_Enabled N -> (none); Spice_Primitive J -> (none)
- J5, J6: Spice_Model PWM -> (none); Spice_Netlist_Enabled N -> (none); Spice_Primitive J -> (none)
- J7: Spice_Model Communication -> (none); Spice_Netlist_Enabled N -> (none); Spice_Primitive J -> (none)
- J8, J9: Spice_Model SJ1-3534N -> (none); Spice_Netlist_Enabled N -> (none); Spice_Primitive J -> (none)
- R15, R18, R19: Spice_Model 7.5k -> (none); Spice_Netlist_Enabled Y -> (none); Spice_Primitive R -> (none)
- R16: Spice_Model 523 -> (none); Spice_Netlist_Enabled Y -> (none); Spice_Primitive R -> (none)
- R17: Spice_Model 11.8k -> (none); Spice_Netlist_Enabled Y -> (none); Spice_Primitive R -> (none)
- U1: Spice_Lib_File CD4066-quad.LIB -> (none); Spice_Model CD4066-quad -> (none); Spice_Netlist_Enabled Y -> (none); Spice_Primitive X -> (none)
- U2: Spice_Lib_File LMC6482-ideal.LIB -> (none); Spice_Model LMC6482 -> (none); Spice_Netlist_Enabled Y -> (none); Spice_Primitive X -> (none)
- V1: Spice_Model dc 3.3 -> (none); Spice_Netlist_Enabled Y -> (none); Spice_Primitive V -> (none)
- V2: Spice_Model dc 0 ac 17.8 sin(0 17.8 60) -> (none); Spice_Netlist_Enabled Y -> (none); Spice_Primitive V -> (none)
- V3: Spice_Model dc 5 -> (none); Spice_Netlist_Enabled Y -> (none); Spice_Primitive V -> (none)
- V4, V6: Spice_Model dc 0 ac 0 pulse(0 5 0 2n 2n 16.667m 33.333m) -> (none); Spice_Netlist_Enabled Y -> (none); Spice_Primitive V -> (none)
- V5, V7: Spice_Model dc 0 ac 0 pulse(0 5 0 2n 2n 16.667m 50m) -> (none); Spice_Netlist_Enabled Y -> (none); Spice_Primitive V -> (none)
